File: wallbox.kicad_pcb (KiCad board)
At the start: 2 copper layers, 166.4 x 94.6 mm, 52 parts, among them J1 From Transformer, J2 To Wallbox, J3 UART, J4 Program, Q1 BC547, Q2 BC547, Q3 BC547, U1 KA78R33, U2 LM7805CT, U3 TPC817MC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

Commit message: Final markings
Parts:
- added G***: LOGO, wallbox-footprints:LogicProbe, F.Cu at (155.6, 99.1)
Other:
- board text added: "Rev: A 2017-10-13"
- board text added: "Wall-O-Matic Interface"
- board text removed: "Rev. A"
- board text removed: "Wall-O-Matic Interface LogicProbe.org"

Commit message: First pass of post-rev-A fixes
Removed Zener diode, that's probably unnecessary and  wasn't working as
intended.
Fixed coin relay connections (25VAC instead of Common)
Tweaked some component labels/values
Parts:
- removed D5: 1N5363, Diodes_THT:D_DO-41_SOD81_P12.70mm_Horizontal
- renumbered Reset to SW1
Connections:
- D1 pad 1: Net-(D1-Pad1) -> Net-(C1-Pad1)
- RL1 pad 7: Net-(D2-Pad2) -> Net-(D1-Pad4)
- RL1 pad 8: Net-(D2-Pad2) -> Net-(D1-Pad4)
- RL2 pad 7: Net-(D2-Pad2) -> Net-(D1-Pad4)
- RL2 pad 8: Net-(D2-Pad2) -> Net-(D1-Pad4)
- RL3 pad 7: Net-(D2-Pad2) -> Net-(D1-Pad4)
- RL3 pad 8: Net-(D2-Pad2) -> Net-(D1-Pad4)
Routing:
- net Net-(D1-Pad4): track 171.7 -> 279.7 mm
- net Net-(D2-Pad2): track 324.2 -> 222.5 mm
- net Net-(C1-Pad1): track 33.3 -> 51.1 mm
- net Net-(D1-Pad1): track 5.08 -> 0.00 mm
Other:
- board text added: "Reset"
- board text added: "Rev: A(?) 2017-10-??"
- board text removed: "Rev: A 2017-10-13"
