File: wallbox.kicad_pcb (KiCad board)
At the start: 2 copper layers, 123.8 x 91.4 mm, 55 parts, among them J1 From Transformer, J2 To Wallbox, J3 UART, J4 Program, Q1 BC547, Q2 BC547, Q3 BC547, SW1 Reset, SW2 Config, U1 KA78R33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

Commit message: Top shrink
Parts:
- moved REF** 7.18 mm to (21.0, 21.0)
- moved REF** 7.18 mm to (137.2, 21.0)
- moved J2 5.08 mm to (128.3, 53.3)
- moved U2 5.08 mm to (74.9, 40.0)
- moved C4 5.08 mm to (64.1, 59.1)
- moved C8 5.08 mm to (47.0, 53.3)
- moved U7 5.08 mm to (67.3, 66.0)
- moved C11 5.08 mm to (26.0, 66.0)
- moved R13 5.08 mm to (29.2, 85.1)
- moved R14 5.08 mm to (29.2, 90.2)
- moved C1 5.08 mm to (54.6, 28.6)
- moved C10 5.08 mm to (32.4, 67.3)
- moved C2 5.08 mm to (76.2, 47.0)
- moved C3 5.08 mm to (69.8, 53.3)
- moved C5 5.08 mm to (80.0, 27.9)
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Routing:
- net Net-(D2-Pad2): track 178.7 -> 160.9 mm
- net Net-(D1-Pad4): track 238.8 -> 221.6 mm, vias 1 -> 0
- net Net-(D2-Pad4): track 93.8 -> 83.6 mm
- net Net-(D1-Pad2): track 95.6 -> 93.8 mm
- net (no net): track 0.00 -> 1.27 mm
- net GND: track 174.2 -> 173.0 mm
Other:
- board size 123.8 x 91.4 mm -> 123.8 x 86.4 mm

Commit message: Routing cleanup
Routing:
- net (no net): track 1.27 -> 0.00 mm
- net Net-(U7-Pad2): track 41.8 -> 41.2 mm
- net Net-(J4-Pad1): track 24.0 -> 23.4 mm
Changed lines of the file:
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@@
     (links 119)
     (no_connects 1)
-    (area 17.094999 16.9796 141.020001 103.7224)
+    (area 17.094999 12.54 150.395715 103.7224)
     (thickness 1.6002)
     (drawings 26)
-    (tracks 444)
+    (tracks 442)
     (zones 0)
     (modules 55)
@@
   )
   (setup
-    (last_trace_width 1.27)
+    (last_trace_width 0.635)
     (user_trace_width 0.254)
     (user_trace_width 0.635)
@@
     (effects (font (size 1.5 1.5) (thickness 0.3)) (justify left))
   )
-  (segment (start 22.86 96.52) (end 21.59 96.52) (width 0.635) (layer B.Cu) (net 0))
   (segment (start 54.61 28.575) (end 57.785 28.575) (width 1.27) (layer B.Cu) (net 1))
   (segment (start 52.07 33.655) (end 52.07 36.83) (width 1.27) (layer B.Cu) (net 1))
@@
   (segment (start 41.91 86.36) (end 41.91 88.9) (width 0.635) (layer F.Cu) (net 18))
   (segment (start 42.29 85.98) (end 41.91 86.36) (width 0.635) (layer F.Cu) (net 18))
-  (segment (start 45.31 86.36) (end 45.69 85.98) (width 0.635) (layer F.Cu) (net 18))
   (segment (start 97.79 29.21) (end 97.79 43.18) (width 0.635) (layer B.Cu) (net 19))
   (segment (start 99.06 44.45) (end 101.6 44.45) (width 0.635) (layer B.Cu) (net 19))
@@
   (segment (start 45.69 83.98) (end 40.48 83.98) (width 0.635) (layer F.Cu) (net 40))
   (segment (start 40.48 83.98) (end 39.37 85.09) (width 0.635) (layer F.Cu) (net 40))
-  (segment (start 69.85 66.04) (end 69.85 68.58) (width 0.635) (layer F.Cu) (net 49))
-  (segment (start 47.91 87.98) (end 45.69 87.98) (width 0.635) (layer F.Cu) (net 49))
-  (segment (start 48.26 87.63) (end 47.91 87.98) (width 0.635) (layer F.Cu) (net 49))
-  (segment (start 48.26 76.835) (end 48.26 87.63) (width 0.635) (layer F.Cu) (net 49))
-  (via (at 48.26 76.835) (size 0.6858) (drill 0.3302) (layers F.Cu B.Cu) (net 49))
-  (segment (start 48.26 75.565) (end 48.26 76.835) (width 0.635) (layer B.Cu) (net 49))
-  (segment (start 49.53 74.295) (end 48.26 75.565) (width 0.635) (layer B.Cu) (net 49))
-  (segment (start 60.96 74.295) (end 49.53 74.295) (width 0.635) (layer B.Cu) (net 49))
-  (via (at 60.96 74.295) (size 0.6858) (drill 0.3302) (layers F.Cu B.Cu) (net 49))
-  (segment (start 66.04 69.215) (end 60.96 74.295) (width 0.635) (layer F.Cu) (net 49))
-  (segment (start 69.215 69.215) (end 66.04 69.215) (width 0.635) (layer F.Cu) (net 49))
-  (segment (start 69.85 68.58) (end 69.215 69.215) (width 0.635) (layer F.Cu) (net 49))
+  (segment (start 47.625 86.045) (end 45.69 87.98) (width 0.635) (layer F.Cu) (net 49))
+  (segment (start 47.625 76.835) (end 47.625 86.045) (width 0.635) (layer F.Cu) (net 49))
+  (segment (start 48.26 76.2) (end 47.625 76.835) (width 0.635) (layer F.Cu) (net 49))
+  (via (at 48.26 76.2) (size 0.6858) (drill 0.3302) (layers F.Cu B.Cu) (net 49))
+  (segment (start 48.26 73.66) (end 48.26 76.2) (width 0.635) (layer B.Cu) (net 49))
+  (via (at 48.26 73.66) (size 0.6858) (drill 0.3302) (layers F.Cu B.Cu) (net 49))
+  (segment (start 48.895 73.025) (end 48.26 73.66) (width 0.635) (layer F.Cu) (net 49))
+  (segment (start 62.23 73.025) (end 48.895 73.025) (width 0.635) (layer F.Cu) (net 49))
+  (segment (start 66.04 69.215) (end 62.23 73.025) (width 0.635) (layer F.Cu) (net 49))
+  (segment (start 68.58 69.215) (end 66.04 69.215) (width 0.635) (layer F.Cu) (net 49))
+  (segment (start 69.85 67.945) (end 68.58 69.215) (width 0.635) (layer F.Cu) (net 49))
+  (segment (start 69.85 66.04) (end 69.85 67.945) (width 0.635) (layer F.Cu) (net 49))
   (segment (start 115.57 29.21) (end 116.84 29.21) (width 1.27) (layer B.Cu) (net 57))
   (segment (start 123.985 43.34) (end 128.27 43.34) (width 1.27) (layer B.Cu) (net 57))
